Commit message: robot modifications made week 5

File: src/mybot_description/urdf/macros.xacro (robot description, xacro)
@@ -1,69 +1,21 @@
 <?xml version="1.0"?>
 <robot>
-  <!--macro name="cylinder_inertia" params="m r h">
-    <inertia  ixx="${m*(3*r*r+h*h)/12}" ixy = "0" ixz = "0"
-      iyy="${m*(3*r*r+h*h)/12}" iyz = "0"
-      izz="${m*r*r/2}"
-    />
-  </macro>
-  <macro name="box_inertia" params="m x y z">
-    <inertia  ixx="${m*(y*y+z*z)/12}" ixy = "0" ixz = "0"
-      iyy="${m*(x*x+z*z)/12}" iyz = "0"
-      izz="${m*(x*x+z*z)/12}"
-    />
-  </macro>
-  <macro name="sphere_inertia" params="m r">
-    <inertia  ixx="${2*m*r*r/5}" ixy = "0" ixz = "0"
-      iyy="${2*m*r*r/5}" iyz = "0"
-      izz="${2*m*r*r/5}"
-    />
-  </macro>
-  <macro name="wheel" params="lr tY">
-    <link name="${lr}_wheel">
-      <collision>
-        <origin xyz="0 0 0" rpy="0 ${PI/2} ${PI/2}" />
-        <geometry>
-          <cylinder length="${wheelWidth}" radius="${wheelRadius}"/>
-        </geometry>
-      </collision>
-      <visual>
-        <origin xyz="0 0 0" rpy="0 ${PI/2} ${PI/2}" />
-        <geometry>
-          <cylinder length="${wheelWidth}" radius="${wheelRadius}"/>
-        </geometry>
-        <material name="black"/>
-      </visual>
-      <inertial>
-        <origin xyz="0 0 0" rpy="0 ${PI/2} ${PI/2}" />
-        <mass value="${wheelMass}"/>
-        <cylinder_inertia m="${wheelMass}" r="${wheelRadius}" h="${wheelWidth}"/>
-      </inertial>
-    </link>
-    <gazebo reference="${lr}_wheel">
-      <mu1 value="1.0"/>
-      <mu2 value="1.0"/>
-      <kp  value="10000000.0" />
-      <kd  value="1.0" />
-      <fdir1 value="1 0 0"/>
-      <material>Gazebo/Black</material>
-    </gazebo>
-    <joint name="${lr}_wheel_hinge" type="continuous">
-      <parent link="chassis"/>
-      <child link="${lr}_wheel"/>
-    <origin xyz="${-wheelPos+chassisLength/2} ${tY*wheelWidth/2+tY*chassisWidth/2} ${wheelRadius}" rpy="0 0 0" />
-      <axis xyz="0 1 0" rpy="0 0 0" />
-      <limit effort="10000" velocity="10000"/>
-      <joint_properties damping="0.0" friction="0.0"/>
-    </joint>
-    <transmission name="${lr}_trans">
-      <type>transmission_interface/SimpleTransmission</type>
-      <joint name="${lr}_wheel_hinge">
-        <hardwareInterface>EffortJointInterface</hardwareInterface>
-      </joint>
-      <actuator name="${lr}Motor">
-        <hardwareInterface>EffortJointInterface</hardwareInterface>
-        <mechanicalReduction>10</mechanicalReduction>
-      </actuator>
-    </transmission>
-  </macro-->
+    <macro name="cylinder_inertia" params="m r h">
+        <inertia  ixx="${m*(3*r*r+h*h)/12}" ixy = "0" ixz = "0"
+            iyy="${m*(3*r*r+h*h)/12}" iyz = "0"
+            izz="${m*r*r/2}"
+            />
+    </macro>
+    <macro name="box_inertia" params="m x y z">
+        <inertia  ixx="${m*(y*y+z*z)/12}" ixy = "0" ixz = "0"
+            iyy="${m*(x*x+z*z)/12}" iyz = "0"
+            izz="${m*(x*x+z*z)/12}"
+            />
+    </macro>
+    <macro name="sphere_inertia" params="m r">
+        <inertia  ixx="${2*m*r*r/5}" ixy = "0" ixz = "0"
+            iyy="${2*m*r*r/5}" iyz = "0"
+            izz="${2*m*r*r/5}"
+            />
+    </macro>
 </robot>

File: src/mybot_description/urdf/mybot.xacro (robot description, xacro)
@@ -1,107 +1,110 @@
 <?xml version='1.0'?>
 <robot name="myrobot" xmlns:xacro="http://www.ros.org/wiki/xacro">
+    <xacro:property name="PI" value="3.1415926535897931"/>
+    <xacro:property name="chassisHeight" value="0.1"/>
+    <xacro:property name="chassisLength" value="0.4"/>
+    <xacro:property name="chassisWidth" value="0.25"/>
+    <xacro:property name="chassisMass" value="50"/>
+    <xacro:property name="casterRadius" value="0.04"/>
+    <xacro:property name="casterMass" value="5"/>
+    <xacro:property name="wheelWidth" value="0.05"/>
+    <xacro:property name="wheelRadius" value="0.08"/>
+    <xacro:property name="wheelPos" value="0.05"/>
+    <xacro:property name="wheelMass" value="5"/>
+    <xacro:property name="cameraSize" value="0.07"/>
+    <xacro:property name="cameraMass" value="0.1"/>
     <xacro:include filename="$(find mybot_description)/urdf/mybot.gazebo" />
     <xacro:include filename="$(find mybot_description)/urdf/materials.xacro" />
     <xacro:include filename="$(find mybot_description)/urdf/macros.xacro" />
-    <xacro:property name="chassisHeight" value="0.1"/>
-    <xacro:property name="chassisLength" value="0.4"/>
-    <xacro:property name="chassisWidth" value="0.2"/>
-    <xacro:property name="chassisMass" value="50"/>
-    <link name='chassis'>
-        <pose>0 0 0.1 0 0 0</pose>
-        <inertial>
-            <mass value="10.0"/>
-            <origin xyz="0.0 0 0.1" rpy=" 0 0 0"/>
-            <inertia
-                ixx="0.5" ixy="0" ixz="0"
-                iyy="1.0" iyz="0"
-                izz="0.1"
-                />
-        </inertial>
-        <collision name='collision'>
+    <link name="footprint" />
+    <joint name="base_joint" type="fixed">
+        <parent link="footprint"/>
+        <child link="chassis"/>
+    </joint>
+    <link name="chassis">
+        <collision>
+            <origin xyz="0 0 ${wheelRadius}" rpy="0 0 0"/>
             <geometry>
                 <box size="${chassisLength} ${chassisWidth} ${chassisHeight}"/>
             </geometry>
         </collision>
-        <visual name='chassis_visual'>
-            <origin xyz="0 0 0" rpy=" 0 0 0"/>
+        <visual>
+            <origin xyz="0 0 ${wheelRadius}" rpy="0 0 0"/>
             <geometry>
-                <box size=".4 .2 .1"/>
+                <box size="${chassisLength} ${chassisWidth} ${chassisHeight}"/>
             </geometry>
-            <material name="green"/>
+            <material name="orange"/>
         </visual>
-        <collision name='caster_collision'>
-            <origin xyz="-0.15 0 -0.05" rpy=" 0 0 0"/>
+        <inertial>
+            <origin xyz="0 0 ${wheelRadius}" rpy="0 0 0"/>
+            <mass value="${chassisMass}"/>
+            <box_inertia m="${chassisMass}" x="${chassisLength}" y="${chassisWidth}" z="${chassisHeight}"/>
+        </inertial>
+    </link>
+    <joint name="fixed" type="fixed">
+        <origin xyz="0 0 ${casterRadius-chassisHeight+wheelRadius}" rpy="0 0 0"/>
+        <parent link="chassis"/>
+        <child link="caster_wheel"/>
+    </joint>
+    <link name="caster_wheel">
+        <collision>
+            <origin xyz="${casterRadius-chassisLength/2} 0 ${casterRadius-chassisHeight+wheelRadius}" rpy="0 0 0"/>
             <geometry>
-                <sphere radius="0.05"/>
+                <sphere radius="${casterRadius}"/>
             </geometry>
-            <surface>
-                <friction>
-                    <ode>
-                        <mu>0</mu>
-                        <mu2>0</mu2>
-                        <slip1>1.0</slip1>
-                        <slip2>1.0</slip2>
-                    </ode>
-                </friction>
-            </surface>
         </collision>
-        <visual name='caster_visual'>
-            <origin xyz="-0.15 0 -0.05" rpy=" 0 0 0"/>
+        <visual>
+            <origin xyz="${casterRadius-chassisLength/2} 0 ${casterRadius-chassisHeight+wheelRadius}" rpy="0 0 0"/>
             <geometry>
-                <sphere radius="0.05"/>
+                <sphere radius="${casterRadius}"/>
             </geometry>
+            <material name="red"/>
         </visual>
+        <inertial>
+            <origin xyz="${casterRadius-chassisLength/2} 0 ${casterRadius-chassisHeight+wheelRadius}" rpy="0 0 0"/>
+            <mass value="${casterMass}"/>
+            <sphere_inertia m="${casterMass}" r="${casterRadius}"/>
+        </inertial>
     </link>
     <link name="left_wheel">
-        <!--origin xyz="0.1 0.13 0.1" rpy="0 1.5707 1.5707"/-->
         <collision name="collision">
-            <origin xyz="0 0 0" rpy="0 1.5707 1.5707"/>
+            <origin xyz="0 0 0" rpy="0 ${PI/2} ${PI/2}"/>
             <geometry>
-                <cylinder radius="0.1" length="0.05"/>
+                <cylinder radius="${wheelRadius}" length="${wheelWidth}"/>
             </geometry>
         </collision>
         <visual name="left_wheel_visual">
-            <origin xyz="0 0 0" rpy="0 1.5707 1.5707"/>
+            <origin xyz="0 0 0" rpy="0 ${PI/2} ${PI/2}"/>
             <geometry>
-                <cylinder radius="0.1" length="0.05"/>
+                <cylinder radius="${wheelRadius}" length="${wheelWidth}"/>
             </geometry>
         </visual>
         <inertial>
-            <origin xyz="0 0 0" rpy="0 1.5707 1.5707"/>
-            <mass value="5"/>
-            <cylinder_inertia m="5" r="0.1" h="0.05"/>
-            <inertia
-                ixx="1.0" ixy="0.0" ixz="0.0"
-                iyy="1.0" iyz="0.0"
-                izz="1.0"/>
+            <origin xyz="0 0 0" rpy="0 ${PI/2} ${PI/2}"/>
+            <mass value="${wheelMass}"/>
+            <cylinder_inertia m="${wheelMass}" r="${wheelRadius}" h="${wheelWidth}"/>
         </inertial>
     </link>
     <link name="right_wheel">
-        <!--origin xyz="0.1 -0.13 0.1" rpy="0 1.5707 1.5707"/-->
         <collision name="collision">
-            <origin xyz="0 0 0" rpy="0 1.5707 1.5707"/>
+            <origin xyz="0 0 0" rpy="0 ${PI/2} ${PI/2}"/>
             <geometry>
-                <cylinder radius="0.1" length="0.05"/>
+                <cylinder radius="${wheelRadius}" length="${wheelWidth}"/>
             </geometry>
         </collision>
         <visual name="right_wheel_visual">
-            <origin xyz="0 0 0" rpy="0 1.5707 1.5707"/>
+            <origin xyz="0 0 0" rpy="0 ${PI/2} ${PI/2}"/>
             <geometry>
-                <cylinder radius="0.1" length="0.05"/>
+                <cylinder radius="${wheelRadius}" length="${wheelWidth}"/>
             </geometry>
         </visual>
         <inertial>
-            <origin xyz="0 0 0" rpy="0 1.5707 1.5707"/>
-            <mass value="5"/>
-            <cylinder_inertia m="5" r="0.1" h="0.05"/>
-            <inertia
-                ixx="1.0" ixy="0.0" ixz="0.0"
-                iyy="1.0" iyz="0.0"
-                izz="1.0"/>
+            <origin xyz="0 0 0" rpy="0 ${PI/2} ${PI/2}"/>
+            <mass value="${wheelMass}"/>
+            <cylinder_inertia m="${wheelMass}" r="${wheelRadius}" h="${wheelWidth}"/>
         </inertial>
     </link>
     <joint type="continuous" name="left_wheel_hinge">
-        <origin xyz="0.1 0.15 0" rpy="0 0 0"/>
+        <origin xyz="${-wheelPos+chassisLength/2} ${wheelWidth/2+chassisWidth/2} ${wheelRadius}" rpy="0 0 0" />
         <child link="left_wheel"/>
         <parent link="chassis"/>
@@ -111,5 +114,5 @@
     </joint>
     <joint type="continuous" name="right_wheel_hinge">
-        <origin xyz="0.1 -0.15 0" rpy="0 0 0"/>
+        <origin xyz="${-wheelPos+chassisLength/2} -${wheelWidth/2+chassisWidth/2} ${wheelRadius}" rpy="0 0 0" />
         <child link="right_wheel"/>
         <parent link="chassis"/>
@@ -119,15 +122,14 @@
     </joint>
     <joint name="hokuyo_joint" type="fixed">
-        <axis xyz="0 1 0" />
-        <origin xyz=".15 0 .1" rpy="0 0 0"/>
+        <axis xyz="0 0 0" />
+        <origin xyz="${chassisLength/2-0.05} 0 ${chassisHeight*2-0.04}" rpy="0 0 0"/>
         <parent link="chassis"/>
         <child link="hokuyo"/>
     </joint>
-    <!-- Hokuyo Laser -->
     <link name="hokuyo">
         <collision>
             <origin xyz="0 0 0" rpy="0 0 0"/>
             <geometry>
-                <box size="0.1 0.1 0.1"/>
+                <box size="${cameraSize} ${cameraSize} ${cameraSize}"/>
             </geometry>
         </collision>
@@ -139,7 +141,7 @@
         </visual>
         <inertial>
-            <mass value="1e-5" />
+            <mass value="${cameraMass}"/>
             <origin xyz="0 0 0" rpy="0 0 0"/>
-            <inertia ixx="1e-6" ixy="0" ixz="0" iyy="1e-6" iyz="0" izz="1e-6" />
+            <box_inertia m="${cameraMass}" x="${cameraSize}" y="${cameraSize}" z="${cameraSize}"/>
         </inertial>
     </link>
